File: KiCAD/avrHVRescueShield2/avrHVRescueShield2/avrHVRescueShield2.kicad_pcb (KiCad board)
At the start: 2 copper layers, 68.6 x 53.3 mm, 24 parts, among them Q1 MUN5311DW1T1G, SW1 SW_Push, U1 ATmega328P-PU, U2 ATtiny85-20PU, U3 ATtiny2313-20PU, U4 MC34063AP

Commit message: schematics n pcb
Parts:
- turned Q1 to 270 degrees
Connections:
- Q1 pad 1: +12V -> GND
- Q1 pad 2: Net-(Q1-Pad2) -> 12V_EN
- Q1 pad 3: Net-(Q1-Pad2) -> 12V_SW
- Q1 pad 4: GND -> +12V
- Q1 pad 5: 12V_EN -> Net-(Q1-Pad5)
- Q1 pad 6: 12V_SW -> Net-(Q1-Pad5)
Routing:
- net DATA6: track 26.9 -> 40.7 mm
- net GND: track 210.4 -> 198.2 mm
- net +5V: track 110.8 -> 120.2 mm
- net ~RESET~: track 104.7 -> 95.6 mm
- net ~WR~: track 46.6 -> 38.8 mm
- net 12V_EN: track 73.7 -> 81.0 mm
- net XA0: track 43.0 -> 49.1 mm
- net XTAL1: track 45.4 -> 39.9 mm
- net RDY: track 50.3 -> 55.6 mm
- net ~GO~: track 24.8 -> 19.6 mm
- net Net-(Q1-Pad5): track 0.00 -> 2.80 mm
- net Net-(Q1-Pad2): track 2.80 -> 0.00 mm
- net DATA7: track 26.9 -> 25.9 mm
- net ~OE~: track 38.7 -> 39.5 mm
- net BS1: track 44.7 -> 44.1 mm
Other:
- board text added: "ardHighVoltageProgrammer-1.1 Design: Jon Sagebrand jonsagebrand@gmail.com github.com/jonsag"
- board text removed: "ardHighVoltageProgrammer Design: Jon Sagebrand jonsagebrand@gmail.com github.com/jonsag"
