File: KiCAD/avrHVRescueShield2/avrHVRescueShield2.kicad_sch (KiCad schematic)
At the start: 24 parts, among them Q1 MUN5311DW1T1G, SW1 SW_Push, U1 ATmega328P-PU, U2 ATtiny85-20PU, U3 ATtiny2313-20PU, U4 MC34063AP

Commit message: error in schematics
Connections:
- net ~{RESET}: now also U1.1 (~{RESET}/PC6); no longer U1.21 (AREF)
Changed lines of the file:
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@@
-    (stroke (width 0) (type default) (color 0 0 0 0))
-  )
-  (wire (pts (xy 33.02 39.37) (xy 35.56 39.37))
     (stroke (width 0) (type default) (color 0 0 0 0))
   )
@@
     (stroke (width 0) (type default) (color 0 0 0 0))
   )
+  (wire (pts (xy 66.04 77.47) (xy 68.58 77.47))
+    (stroke (width 0) (type default) (color 0 0 0 0))
+  )
   (wire (pts (xy 134.62 59.69) (xy 132.08 59.69))
     (stroke (width 0) (type default) (color 0 0 0 0))
@@
     )
   )
-  (global_label "~{RESET}" (shape input) (at 33.02 39.37 180) (fields_autoplaced)
-    (effects (font (size 1.27 1.27)) (justify right))
-    (property "Intersheet References" "${INTERSHEET_REFS}" (id 0) (at 0 0 0)
-      (effects (font (size 1.27 1.27)) hide)
-    )
-  )
   (global_label "~{WR}" (shape input) (at 68.58 90.17 0) (fields_autoplaced)
     (effects (font (size 1.27 1.27)) (justify left))
@@
       (effects (font (size 1.27 1.27)) hide)
     )
+  )
+  (global_label "~{RESET}" (shape input) (at 68.58 77.47 0) (fields_autoplaced)
+    (effects (font (size 1.27 1.27)) (justify left))
+    (property "Intersheet References" "${INTERSHEET_REFS}" (id 0) (at 101.6 116.84 0)
+      (effects (font (size 1.27 1.27)) hide)
+    )

Commit message: new PCB
Parts:
- added R5: 1R, My_Misc:R_Axial_DIN0207_L6.3mm_D2.5mm_P10.16mm_Horizontal_large, symbol Device:R
- added R6: 1k, My_Misc:R_Axial_DIN0207_L6.3mm_D2.5mm_P10.16mm_Horizontal_large, symbol Device:R
- added TP1: +12V, My_Misc:Single_solder_pad, symbol Connector:TestPoint
- added TP2: 12V EN, My_Misc:Single_solder_pad, symbol Connector:TestPoint
- added TP4: +5V, My_Misc:Single_solder_pad, symbol Connector:TestPoint
- added TP5: GND, My_Misc:Single_solder_pad, symbol Connector:TestPoint
- R1: footprint My_Misc:R_Axial_DIN0207_L6.3mm_D2.5mm_P10.16mm_Horizontal_larger_pads -> My_Misc:R_Axial_DIN0207_L6.3mm_D2.5mm_P10.16mm_Horizontal_large
- R10: renamed from R8; footprint My_Misc:R_Axial_DIN0207_L6.3mm_D2.5mm_P10.16mm_Horizontal_larger_pads -> My_Misc:R_Axial_DIN0207_L6.3mm_D2.5mm_P10.16mm_Horizontal_large
- R2: value 0.5R -> 1R; footprint My_Misc:R_Axial_DIN0207_L6.3mm_D2.5mm_P10.16mm_Horizontal_larger_pads -> My_Misc:R_Axial_DIN0207_L6.3mm_D2.5mm_P10.16mm_Horizontal_large
- R3: renamed from R4; value 13k -> 12k; footprint My_Misc:R_Axial_DIN0207_L6.3mm_D2.5mm_P10.16mm_Horizontal_larger_pads -> My_Misc:R_Axial_DIN0207_L6.3mm_D2.5mm_P10.16mm_Horizontal_large
- R4: renamed from R3; footprint My_Misc:R_Axial_DIN0207_L6.3mm_D2.5mm_P10.16mm_Horizontal_larger_pads -> My_Misc:R_Axial_DIN0207_L6.3mm_D2.5mm_P10.16mm_Horizontal_large
- R7: renamed from R6; footprint My_Misc:R_Axial_DIN0207_L6.3mm_D2.5mm_P10.16mm_Horizontal_larger_pads -> My_Misc:R_Axial_DIN0207_L6.3mm_D2.5mm_P10.16mm_Horizontal_large
- R8: renamed from R7; footprint My_Misc:R_Axial_DIN0207_L6.3mm_D2.5mm_P10.16mm_Horizontal_larger_pads -> My_Misc:R_Axial_DIN0207_L6.3mm_D2.5mm_P10.16mm_Horizontal_large
- R9: renamed from R5; footprint My_Misc:R_Axial_DIN0207_L6.3mm_D2.5mm_P10.16mm_Horizontal_larger_pads -> My_Misc:R_Axial_DIN0207_L6.3mm_D2.5mm_P10.16mm_Horizontal_large
- TP3: renamed from TP1; value TestPoint -> 12V SW
- U1: footprint Package_DIP:DIP-28_W7.62mm_Socket_LongPads -> My_Misc:ZIF_DIP_Socket-28_W6.9_W7.62_W7.62_W12.7_W13.5_large
- U3: footprint Package_DIP:DIP-20_W7.62mm_Socket_LongPads -> My_Misc:ZIF_DIP_Socket-20_W4.3_W5.08_W7.62_W10.16_W10.9_3M_220-3342-00-0602J_large
Connections:
- net +12V: now also R6.2, TP1.1; no longer R3.1
- net +5V: now also R5.1, TP4.1
- net 12V_EN: now also TP2.1
- net GND: now also TP5.1
- net at L1.1, R2.2, R4.1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: now also R5.2
- new net: R3.1, R6.1
Other:
- moved on the sheet: R3
