File: KiCAD/avrHVRescueShield2-smd/avrHVRescueShield2-smd.kicad_pcb (KiCad board)
At the start: 2 copper layers, 69.8 x 54.6 mm, 24 parts, among them Q1 MUN5311DW1T1G, SW1 SW_Push, U1 ATmega328P-PU, U2 ATtiny85-20PU, U3 ATtiny2313-20PU, U4 MC34063AP

Commit message: kicad
Other:
- board text added: "avrHVRescueShield Design: Jon Sagebrand github.com/jonsag/ardHighVoltageProgrammer"
- board text removed: "${TITLE}-${REVISION} Design: Jon Sagebrand github.com/jonsag/ardHighVoltageProgrammer"
Changed lines of the file:
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@@
   )
   (paper "A4")
-  (title_block
-    (title "avrHVRescueShield2")
-    (date "2022-09-09")
-    (rev "1.1")
-  )
   (layers
     (0 "F.Cu" signal)
@@
   (gr_line (start 172.085 75.565) (end 172.085 64.135) (layer "Edge.Cuts") (width 0.05))
   (gr_line (start 104.775 62.23) (end 104.775 116.84) (layer "Edge.Cuts") (width 0.05))
-  (gr_text "${TITLE}-${REVISION}\nDesign: Jon Sagebrand\ngithub.com/jonsag/ardHighVoltageProgrammer" (at 131.445 105.41 90) (layer "F.SilkS")
+  (gr_text "avrHVRescueShield\nDesign: Jon Sagebrand\ngithub.com/jonsag/ardHighVoltageProgrammer" (at 131.445 105.41 90) (layer "F.SilkS")
     (effects (font (size 0.635 0.635) (thickness 0.127)) (justify left))
   )
