File: KiCAD/avrHVRescueShield2-smd/avrHVRescueShield2-smd.kicad_sch (KiCad schematic)
At the start: 24 parts, among them Q1 MUN5311DW1T1G, SW1 SW_Push, U1 ATmega328P-PU, U2 ATtiny85-20PU, U3 ATtiny2313-20PU, U4 MC34063AP

Commit message: kicad
Parts:
- C1: footprint My_Misc:CP_Radial_D5.0mm_P2.50mm_larger_pads -> Capacitor_SMD:CP_Elec_8x10
- C2, C4: footprint My_Misc:C_Disc_D3.0mm_W1.6mm_P2.50mm_larg -> Capacitor_SMD:C_1206_3216Metric_Pad1.33x1.80mm_HandSolder
- C3: footprint My_Misc:CP_Radial_D10.0mm_P5.00mm_larger -> Capacitor_SMD:CP_Elec_10x10
- D1: footprint My_Misc:D_DO-35_SOD27_P7.62mm_Horizontal_large -> Diode_SMD:D_SMC_Handsoldering
- D2, D3: footprint My_Misc:LED_D5.0mm_larger_pads -> LED_SMD:LED_1206_3216Metric_Pad1.42x1.75mm_HandSolder
- L1: footprint My_Misc:L_Axial_L9.5mm_D4.0mm_P12.70mm_Horizontal_Fastron_SMCC_large -> Inductor_SMD:L_1210_3225Metric_Pad1.42x2.65mm_HandSolder
- R1, R2, R3, R4, R5, R6, R7, R8: footprint My_Misc:R_Axial_DIN0207_L6.3mm_D2.5mm_P10.16mm_Horizontal_larger_pads -> Resistor_SMD:R_1206_3216Metric_Pad1.30x1.75mm_HandSolder
Other:
- title: avrHVRescueShield2 -> (none)
