File: KiCAD/ISP_Fuse_Rescue/ISP_Fuse_Rescue.kicad_sch (KiCad schematic)
At the start: 18 parts, among them Q1 2N5551, Q2 2N5551, SW2 SW_Push

Commit message: ISP Fuse Rescue
Parts:
- added H1, H2, H3, H4: MountingHole, MountingHole:MountingHole_3.2mm_M3, symbol Mechanical:MountingHole
- A1: footprint PCM_arduino-library:Arduino_Uno_R3_Shield -> My_Arduino:Arduino_UNO_R3_shield_incl ICSP_headers_large
- D1, D2, D3, D4, D5, D6: footprint (none) -> My_Misc:LED_D5.0mm_large
- Q1, Q2: footprint Package_TO_SOT_THT:TO-92_Inline -> My_Misc:TO-92_Inline_Wide_large
- R1: renamed from R2; footprint (none) -> My_Misc:R_Axial_DIN0207_L6.3mm_D2.5mm_P10.16mm_Horizontal_large
- R2: renamed from R3; footprint (none) -> My_Misc:R_Axial_DIN0207_L6.3mm_D2.5mm_P10.16mm_Horizontal_large
- R3: renamed from R1; footprint (none) -> My_Misc:R_Axial_DIN0207_L6.3mm_D2.5mm_P10.16mm_Horizontal_large
- R4, R5, R6, R7, R8: footprint (none) -> My_Misc:R_Axial_DIN0207_L6.3mm_D2.5mm_P10.16mm_Horizontal_large
- SW1: renamed from SW2; value SW_Push -> Reset; footprint (none) -> My_Misc:SW_PUSH_6mm_large
Other:
- added sheet ATMega328P (atmega328p.kicad_sch)
