File: KiCAD/ISP_Fuse_Rescue SMD/ISP_Fuse_Rescue SMD.kicad_sch (KiCad schematic)
At the start: 22 parts, among them Q1 MMBT3904, Q2 MMBT3904, SW1 Reset

Commit message: smd fuse rescue
Parts:
- removed H1, H2, H3, H4: MountingHole, MountingHole:MountingHole_3.2mm_M3, symbol Mechanical:MountingHole
